File: Hardware/Koroliov_SSDV/Koroliov_v2.sch (EAGLE design)
At the start: 24 parts

Commit message: Fixes after first fabrication
Arduino Micro was not fully compatible with previous layout for the
camera and the SD card. Antenna SMA connector has been moved to edge for
better connection with antenna cable.
Parts:
- removed ANTENNA: BU-SMA-V, con-coax:BU-SMA-V
- added ANT: (no value), adafruit:SMACONNECTOR_EDGE
Connections:
- new net STATUS_SD: ARDUINOMICRO.13
- net CAMTX: now also ARDUINOMICRO.8; no longer ARDUINOMICRO.4
- net GND: now also ANT.GND1, ANT.GND2, ANT.GND3, ANT.GND4; no longer ANTENNA.2
- net N$1: now also ANT.ANT; no longer ANTENNA.1
- net SDCLK: now also ARDUINOMICRO.SCK; no longer ARDUINOMICRO.13
- net SDDI: now also ARDUINOMICRO.MOSI; no longer ARDUINOMICRO.11
- net SDDO: now also ARDUINOMICRO.MISO; no longer ARDUINOMICRO.12
- net STATUS_RADIO: now also ARDUINOMICRO.4; no longer ARDUINOMICRO.8
